Commit message: renamed flexicart macro for srdf

File: ilab_franka_description/srdf/flexicart.xacro (robot description, xacro)
@@ -1,5 +1,5 @@
 <?xml version="1.0" ?>
 <robot xmlns:xacro="http://www.ros.org/wiki/xacro" name="franka">
-  <xacro:macro name="flexicart" params="arm_id:='franka' ">
+  <xacro:macro name="franka_flexicart" params="arm_id:='franka' ">
     <disable_collisions link1="${arm_id}_flexicart" link2="${arm_id}_link0" reason="Adjacent"/>
     <disable_collisions link1="${arm_id}_flexicart" link2="${arm_id}_link1" reason="Adjacent"/>

File: ilab_franka_description/srdf/ilab_franka.srdf.xacro (robot description, xacro)
@@ -5,5 +5,5 @@
   <xacro:property name="arm_id" value="$(arg arm_id)"/>
   <xacro:include filename="$(find ilab_franka_description)/srdf/flexicart.xacro"/>
-  <xacro:flexicart arm_id="${arm_id}"/>
+  <xacro:franka_flexicart arm_id="${arm_id}"/>
   <xacro:include filename="$(find ilab_franka_description)/srdf/franka_arm.xacro"/>
   <xacro:franka_arm arm_id="${arm_id}"/>
